Commit message: new shelf moveit package

File: config/gazebo_ur5e_robot.urdf (robot description, URDF)
Before this commit: robot ur5e_robot, 22 links, 21 joints
Links:
- link stand_link: geometry collision box size=1.08 1.08 0.9; visual box size=1.08 1.08 0.9
Joints:
- joint realsense_link: origin xyz=0.025 -0.065 -0.02 rpy=0 0 0 -> xyz=-0.025 0.065 -0.02 rpy=0 0 0
- joint shelf_joint: origin xyz=0 -0.5 0 rpy=0 0 3.14 -> xyz=0 -0.54 0 rpy=1.57 0 3.14
